File: 6502-pcbs/6502-pcbs.kicad_pcb (KiCad board)
At the start: 0 parts

Commit message: datasheets and bus timing
Parts:
- added C3: 1uF, Capacitor_THT:CP_Axial_L10.0mm_D4.5mm_P15.00mm_Horizontal, F.Cu at (186.4, 49.0)
- added C4: 0.1uF, Capacitor_THT:CP_Radial_D4.0mm_P1.50mm, F.Cu at (170.6, 36.5)
- added C5: 0.1uF, Capacitor_THT:CP_Radial_D4.0mm_P1.50mm, F.Cu at (170.6, 42.1)
- added C6: 0.01uF, Capacitor_THT:CP_Radial_D4.0mm_P1.50mm, F.Cu at (170.6, 47.6)
- added C7: 0.01uF, Capacitor_THT:CP_Radial_D4.0mm_P1.50mm, F.Cu at (170.6, 53.2)
- added C8: 0.1uF, Capacitor_THT:CP_Radial_D4.0mm_P1.50mm, F.Cu at (170.6, 58.7)
- added C9: 0.01uF, Capacitor_THT:CP_Radial_D4.0mm_P1.50mm, F.Cu at (170.6, 64.3)
- added D1: RED, LED_THT:LED_D5.0mm_Horizontal_O6.35mm_Z9.0mm, F.Cu at (101.3, 133.7)
- added D3: YELLOW, LED_THT:LED_D5.0mm_Horizontal_O6.35mm_Z9.0mm, F.Cu at (108.8, 133.7)
- added D4: YELLOW, LED_THT:LED_D5.0mm_Horizontal_O6.35mm_Z9.0mm, F.Cu at (116.2, 133.7)
- added D5: YELLOW, LED_THT:LED_D5.0mm_Horizontal_O6.35mm_Z9.0mm, F.Cu at (123.7, 133.7)
- added D6: YELLOW, LED_THT:LED_D5.0mm_Horizontal_O6.35mm_Z9.0mm, F.Cu at (131.2, 133.7)
- added R1: 1k, Resistor_THT:R_Axial_DIN0309_L9.0mm_D3.2mm_P12.70mm_Horizontal, F.Cu at (84.5, 81.9)
- added R10: 220, Resistor_THT:R_Axial_DIN0309_L9.0mm_D3.2mm_P12.70mm_Horizontal, F.Cu at (84.5, 124.7)
- added R11: 220, Resistor_THT:R_Axial_DIN0309_L9.0mm_D3.2mm_P12.70mm_Horizontal, F.Cu at (84.5, 129.4)
- added R12: 1k, Resistor_THT:R_Axial_DIN0309_L9.0mm_D3.2mm_P12.70mm_Horizontal, F.Cu at (84.5, 134.2)
- added R13: 220, Resistor_THT:R_Axial_DIN0309_L9.0mm_D3.2mm_P12.70mm_Horizontal, F.Cu at (84.5, 138.9)
- added R2: 1k, Resistor_THT:R_Axial_DIN0309_L9.0mm_D3.2mm_P12.70mm_Horizontal, F.Cu at (84.5, 86.7)
- added R3: 1k, Resistor_THT:R_Axial_DIN0309_L9.0mm_D3.2mm_P12.70mm_Horizontal, F.Cu at (84.5, 91.4)
- added R4: 1M, Resistor_THT:R_Axial_DIN0309_L9.0mm_D3.2mm_P12.70mm_Horizontal, F.Cu at (84.5, 96.2)
- added R5: 1k, Resistor_THT:R_Axial_DIN0309_L9.0mm_D3.2mm_P12.70mm_Horizontal, F.Cu at (84.5, 100.9)
- added R6: 1k, Resistor_THT:R_Axial_DIN0309_L9.0mm_D3.2mm_P12.70mm_Horizontal, F.Cu at (84.5, 105.7)
- added R7: 1k, Resistor_THT:R_Axial_DIN0309_L9.0mm_D3.2mm_P12.70mm_Horizontal, F.Cu at (84.5, 110.4)
- added R8: 220, Resistor_THT:R_Axial_DIN0309_L9.0mm_D3.2mm_P12.70mm_Horizontal, F.Cu at (84.5, 115.2)
- added R9: 220, Resistor_THT:R_Axial_DIN0309_L9.0mm_D3.2mm_P12.70mm_Horizontal, F.Cu at (84.5, 119.9)
- added RV1: 10k?, Potentiometer_THT:Potentiometer_Bourns_3386C_Horizontal, F.Cu at (187.9, 55.0)
- added RV2: 1M, Potentiometer_THT:Potentiometer_Bourns_3386C_Horizontal, F.Cu at (194.3, 55.0)
- added SW1: Push, Button_Switch_THT:SW_PUSH_6mm, F.Cu at (176.1, 47.5)
- added SW2: Push, Button_Switch_THT:SW_PUSH_6mm, F.Cu at (176.1, 56.0)
- added SW3: SW_SPDT, Button_Switch_SMD:SW_SPDT_PCM12, F.Cu at (202.4, 54.9)
- added SW4: Push, Button_Switch_THT:SW_PUSH_6mm, F.Cu at (176.1, 64.6)
- added U1: W65C02SxP, Package_DIP:DIP-40_W15.24mm, F.Cu at (100.4, 81.6)
- added U10: 74LS08, Package_DIP:DIP-14_W7.62mm, F.Cu at (155.6, 118.7)
- added U11: 74LS04, Package_DIP:DIP-14_W7.62mm, F.Cu at (166.4, 118.7)
- added U12: 74LS32, Package_DIP:DIP-14_W7.62mm, F.Cu at (177.1, 118.7)
- added U13: ATmega644-20P, Package_DIP:DIP-40_W15.24mm, F.Cu at (137.2, 81.6)
- added U14: 74HC00, Package_DIP:DIP-14_W7.62mm, F.Cu at (187.9, 118.7)
- added U2: HM62256BLP, Package_DIP:DIP-28_W15.24mm, F.Cu at (155.6, 81.6)
- added U3: 28C256, Package_DIP:DIP-28_W15.24mm, F.Cu at (174.0, 81.6)
- added U4: W65C22SxP, Package_DIP:DIP-40_W15.24mm, F.Cu at (118.8, 81.6)
- added U5: RC1602A, Display:RC1602A, F.Cu at (124.5, 36.8)
- added U6: W65C51NxP, Package_DIP:DIP-28_W15.24mm, F.Cu at (192.3, 81.6)
- added U7: NE555P, Package_DIP:DIP-8_W7.62mm, F.Cu at (175.7, 35.8)
- added U8: NE555P, Package_DIP:DIP-8_W7.62mm, F.Cu at (186.5, 35.8)
- added U9: NE555P, Package_DIP:DIP-8_W7.62mm, F.Cu at (197.3, 35.8)
Other:
- copper layers 0 -> 2
