File: 6502-pcbs/555-clock/555-clock.kicad_sch (KiCad schematic)
At the start: 0 parts

Commit message: 555-clock
Parts:
- added C3: 1uF, Capacitor_THT:CP_Axial_L10.0mm_D4.5mm_P15.00mm_Horizontal, symbol Device:C_Small_US
- added C4, C5, C8: 0.1uF, Capacitor_THT:CP_Radial_D4.0mm_P1.50mm, symbol Device:C_Small
- added C6, C7, C9: 0.01uF, Capacitor_THT:CP_Radial_D4.0mm_P1.50mm, symbol Device:C_Small
- added D1, D3, D4, D5: YELLOW, LED_THT:LED_D5.0mm_Horizontal_O6.35mm_Z9.0mm, symbol Device:LED
- added D6: RED, LED_THT:LED_D5.0mm_Horizontal_O6.35mm_Z9.0mm, symbol Device:LED
- added J1: Universal Bus Connector, symbol Connector_Generic:Conn_02x20_Odd_Even
- added J2: Halt Clk, symbol Connector_Generic:Conn_01x02
- added R10, R11, R13, R8, R9: 220, Resistor_THT:R_Axial_DIN0309_L9.0mm_D3.2mm_P12.70mm_Horizontal, symbol Device:R_Small_US
- added R2, R3, R5, R6, R7: 1k, Resistor_THT:R_Axial_DIN0309_L9.0mm_D3.2mm_P12.70mm_Horizontal, symbol Device:R_Small_US
- added R4: 1M, Resistor_THT:R_Axial_DIN0309_L9.0mm_D3.2mm_P12.70mm_Horizontal, symbol Device:R_Small_US
- added RV2: 1M, Potentiometer_THT:Potentiometer_Bourns_3386C_Horizontal, symbol Device:R_Potentiometer_US
- added SW2: Push, Button_Switch_THT:SW_PUSH_6mm, symbol Switch:SW_Push
- added SW3: SW_SPDT, Button_Switch_SMD:SW_SPDT_PCM12, symbol Switch:SW_SPDT
- added U10: 74LS08, Package_DIP:DIP-14_W7.62mm, symbol 74xx:74LS08
- added U11: 74LS04, Package_DIP:DIP-14_W7.62mm, symbol 74xx:74LS04
- added U12: 74LS32, Package_DIP:DIP-14_W7.62mm, symbol 74xx:74LS32
- added U7, U8, U9: NE555P, Package_DIP:DIP-8_W7.62mm, symbol Timer:NE555P
Connections:
- new net: D1.1 (K), R8.1
- new net: D4.1 (K), R10.1
- new net: D5.1 (K), R11.1
- new net: D5.2 (A), U10.2, U11.1, U9.3 (Q)
- new net: U10.3, U12.1
- new net: U10.6, U12.2
- new net: U10.9, U12.3
- new net: C6.1, U7.5 (CV)
- new net: C3.1, RV2.3, U7.2 (TR), U7.6 (THR)
- new net: D4.2 (A), U10.1, U7.3 (Q)
- new net: R2.2, R3.1, U7.7 (DIS)
- new net: J2.1 (Pin_1), U10.10
- new net: D1.2 (A), J1.30 (Pin_30), U10.8
- new net: R6.2, SW3.1 (A), U9.2 (TR)
- new net: D6.1 (K), R13.1
- new net: J1.32 (Pin_32), U11.3
- new net: D6.2 (A), J2.2 (Pin_2), U11.4
- new net: C9.1, U9.5 (CV)
- new net: R5.2, SW2.2, U8.2 (TR)
- new net: R3.2, RV2.2
- new net: D3.2 (A), U10.5, U8.3 (Q)
- new net: C7.1, U8.5 (CV)
- new net: C8.1, R4.2, U8.6 (THR), U8.7 (DIS)
- new net: R7.2, SW3.3 (C), U9.4 (R)
- new net: U10.4, U11.2
- new net: D3.1 (K), R9.1
- new net +5V: C4.1, C5.1, J1.3 (Pin_3), J1.37 (Pin_37), J1.38 (Pin_38), J1.4 (Pin_4), R2.1, R4.1, R5.1, U7.4 (R), U7.8 (VCC), U8.4 (R), U8.8 (VCC)
- new net GND: C3.2, C4.2, C5.2, C6.2, C7.2, C8.2, C9.2, J1.1 (Pin_1), J1.2 (Pin_2), J1.39 (Pin_39), J1.40 (Pin_40), R10.2, R11.2, R13.2, R8.2, R9.2, SW2.1, SW3.2 (B), U7.1 (GND), U8.1 (GND), U9.1 (GND), U9.6 (THR)
- no-connect marks 0 -> 32
