File: 6502-pcbs/full-schematic/full-schematic.kicad_sch (KiCad schematic)
At the start: 47 parts, among them SW1 Push, SW2 Push, SW3 SW_SPDT, SW4 SW_SPDT, U1 W65C02SxP, U10 74LS08, U11 74LS04, U12 74LS32, U13 ATmega644-20P, U14 74HC00, U15 74HC00, U16 74HC00, U2 HM62256BLP, U3 28C256, U4 W65C22SxP, U5 RC1602A, U6 W65C51NxP, U7 NE555P, U8 NE555P, U9 NE555P, Y1 ACO-xxxMHz

Commit message: 555-clock
Parts:
- added J1: Halt CLK, symbol Connector_Generic:Conn_01x02
- D1: value RED -> YELLOW
- D6: value YELLOW -> RED
Connections:
- net +5V: no longer U1.2 (RDY), U1.36 (BE)
- net at U1.7 (SYNC): now also U13.20 (PD6)
- net at U13.19 (PD5): now also U1.36 (BE)
- net at U11.4: now also D6.2 (A), J1.2 (Pin_2); no longer U10.10
- net HALT: no longer names the net of U11.3, U13.14 (PD0)
- net HALT: now also U1.2 (RDY); no longer D6.2 (A)
- new net: J1.1 (Pin_1), U10.10
- no-connect marks 24 -> 21

Commit message: 6502 mainboard
Parts:
- removed SW4: SW_SPDT, Button_Switch_SMD:SW_SPDT_PCM12, symbol Switch:SW_SPDT
- added C1: 10uF+, symbol Device:C_Polarized_Small
- added C10, C11, C12, C13, C14, C15, C16, C17, C18, C2: 100nF, symbol Device:C_Small
- added D2: YELLOW, LED_THT:LED_D5.0mm_Horizontal_O6.35mm_Z9.0mm, symbol Device:LED
- added J2: 1MHz CLK, symbol Connector_Generic:Conn_01x02
- added J3: Barrel_Jack, symbol Connector:Barrel_Jack
- added R12: 220, Resistor_THT:R_Axial_DIN0309_L9.0mm_D3.2mm_P12.70mm_Horizontal, symbol Device:R_Small_US
- C4, C5: value 0.1uF -> 100nF; footprint Capacitor_THT:CP_Radial_D4.0mm_P1.50mm -> (none)
Connections:
- net +5V: now also U6.15 (VCC), C1.1, C10.1, C11.1, C12.1, C13.1, C14.1, C15.1, C16.1, C17.1, C18.1, C2.1, D2.2 (A), J3.1
- net GND: now also C1.2, C10.2, C11.2, C12.2, C13.2, C14.2, C15.2, C16.2, C17.2, C18.2, C2.2, J3.2, R12.2
- net at D1.2 (A), U10.8, U11.5: now also U1.37 (ϕ0), U13.16 (PD2), U16.2, U4.25 (ϕ2), J2.2 (Pin_2)
- net at Y1.8 (OUT): now also J2.1 (Pin_1)
- new net: D2.1 (K), R12.1

Commit message: 28c256 rom
Other:
- company: (none) -> Sam Warr
- title: (none) -> 6502 Stacked
- moved on the sheet: C1, C10, C11, C12, C13, C14, C15, C16, C17, C18, C2, C3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
