File: 6502-pcbs/28c256-rom/28c256-rom.kicad_pcb (KiCad board)
At the start: 0 parts

Commit message: 28c256 rom pcb
Parts:
- added C15: 100nF, Capacitor_THT:C_Rect_L4.6mm_W2.0mm_P2.50mm_MKS02_FKP02, F.Cu at (151.8, 46.0)
- added C7: 100nF, Capacitor_THT:C_Rect_L4.6mm_W2.0mm_P2.50mm_MKS02_FKP02, F.Cu at (124.1, 36.9)
- added C8: 100nF, Capacitor_THT:C_Rect_L4.6mm_W2.0mm_P2.50mm_MKS02_FKP02, F.Cu at (93.5, 83.1)
- added J3: Universal Bus Connector A, Connector_PinSocket_2.54mm:PinSocket_1x18_P2.54mm_Vertical, F.Cu at (126.6, 40.0)
- added J4: Universal Bus Connector B, Connector_PinSocket_2.54mm:PinSocket_1x18_P2.54mm_Vertical, F.Cu at (126.6, 80.0)
- added U14: 74HC00, Package_DIP:DIP-14_W7.62mm, F.Cu at (144.3, 49.2)
- added U3: 28C256, Package_DIP:DIP-28_W15.24mm, F.Cu at (89.1, 67.4)
Routing:
- net +5V: track 0.00 -> 183.0 mm
- net Net-(J3-Pin_18): track 0.00 -> 112.3 mm
- net Net-(J4-Pin_6): track 0.00 -> 91.6 mm
- net Net-(J4-Pin_2): track 0.00 -> 86.3 mm
- net Net-(J4-Pin_7): track 0.00 -> 80.0 mm
- net Net-(J4-Pin_8): track 0.00 -> 76.4 mm
- net Net-(J4-Pin_9): track 0.00 -> 72.8 mm
- net Net-(J4-Pin_10): track 0.00 -> 69.2 mm
- net Net-(J3-Pin_10): track 0.00 -> 68.8 mm
- net Net-(J3-Pin_9): track 0.00 -> 65.3 mm
- net Net-(J3-Pin_8): track 0.00 -> 61.7 mm
- net Net-(J3-Pin_7): track 0.00 -> 58.1 mm
- net Net-(J3-Pin_6): track 0.00 -> 54.6 mm
- net Net-(J3-Pin_5): track 0.00 -> 51.1 mm
- net Net-(J3-Pin_4): track 0.00 -> 47.6 mm
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- added copper zone on B.Cu, net GND
Other:
- board outline added: 100 x 70 mm
- copper layers 0 -> 2
