File: 6502-pcbs/28c256-rom/28c256-rom.kicad_sch (KiCad schematic)
At the start: 0 parts

Commit message: 28c256 rom
Parts:
- added C15: 100nF, symbol Device:C_Small
- added C7: 100nF, Capacitor_THT:C_Rect_L4.6mm_W2.0mm_P2.50mm_MKS02_FKP02, symbol Device:C_Small
- added J3, J4: Universal Bus Connector v2, symbol Connector:Conn_01x18_Socket
- added U14: 74HC00, Package_DIP:DIP-14_W7.62mm, symbol 74xx:74HC00
- added U3: 28C256, Package_DIP:DIP-28_W15.24mm, symbol Memory_EEPROM:28C256
Connections:
- new net: J4.10 (Pin_10), U3.19 (D7)
- new net: J4.3 (Pin_3), U3.11 (D0)
- new net: J4.4 (Pin_4), U3.12 (D1)
- new net: J4.5 (Pin_5), U3.13 (D2)
- new net: J4.6 (Pin_6), U3.15 (D3)
- new net: J4.7 (Pin_7), U3.16 (D4)
- new net: J4.8 (Pin_8), U3.17 (D5)
- new net: J4.9 (Pin_9), U3.18 (D6)
- new net: J3.10 (Pin_10), U3.3 (A7)
- new net: J3.11 (Pin_11), U3.25 (A8)
- new net: J3.12 (Pin_12), U3.24 (A9)
- new net: J3.13 (Pin_13), U3.21 (A10)
- new net: J3.14 (Pin_14), U3.23 (A11)
- new net: J3.15 (Pin_15), U3.2 (A12)
- new net: J3.16 (Pin_16), U3.26 (A13)
- new net: J3.3 (Pin_3), U3.10 (A0)
- new net: J3.4 (Pin_4), U3.9 (A1)
- new net: J3.5 (Pin_5), U3.8 (A2)
- new net: J3.6 (Pin_6), U3.7 (A3)
- new net: J3.7 (Pin_7), U3.6 (A4)
- new net: J3.8 (Pin_8), U3.5 (A5)
- new net: J3.9 (Pin_9), U3.4 (A6)
- new net: U14.3, U3.20 (~{CS})
- new net +5V: C15.1, C7.1, J3.2 (Pin_2), J4.2 (Pin_2), U3.28 (VCC)
- new net GND: C15.2, C7.2, J3.1 (Pin_1), J4.1 (Pin_1), U3.14 (GND), U3.22 (~{OE})
- no-connect marks 0 -> 6
Other:
- company: (none) -> Sam Warr
- title: (none) -> 28C256 ROM Board

Commit message: 28c256 rom pcb
Parts:
- added C8: 100nF, Capacitor_THT:C_Rect_L4.6mm_W2.0mm_P2.50mm_MKS02_FKP02, symbol Device:C_Small
- added unit 3 of U14
- added unit 2 of U14
- added unit 5 of U14
- added unit 4 of U14
- C15: footprint (none) -> Capacitor_THT:C_Rect_L4.6mm_W2.0mm_P2.50mm_MKS02_FKP02
- J3: value Universal Bus Connector v2 -> Universal Bus Connector A; footprint (none) -> Connector_PinSocket_2.54mm:PinSocket_1x18_P2.54mm_Vertical
- J4: value Universal Bus Connector v2 -> Universal Bus Connector B; footprint (none) -> Connector_PinSocket_2.54mm:PinSocket_1x18_P2.54mm_Vertical
Connections:
- net +5V: now also J4.13 (Pin_13), C8.2, U14.14 (VCC); no longer J4.2 (Pin_2)
- net GND: now also J4.14 (Pin_14), C8.1, U14.10, U14.12, U14.13, U14.4, U14.5, U14.7 (GND), U14.9; no longer J4.1 (Pin_1)
- net at J3.17 (Pin_17): now also U3.1 (A14)
- net at J3.18 (Pin_18): now also U14.1, U14.2
- net at U3.27 (~{WE}): now also J4.2 (Pin_2)
- no-connect marks 6 -> 10
Other:
- moved on the sheet: C15, C7, J3, J4, U14A, U3
