File: 6502-pcbs/6502-mainboard/6502-mainboard.kicad_pcb (KiCad board)
At the start: 0 parts

Commit message: 6502 mainboard
Parts:
- added C1: 10uF+, Capacitor_THT:CP_Radial_D7.5mm_P2.50mm, F.Cu at (144.3, 41.0)
- added C13: 100nF, Capacitor_THT:C_Rect_L4.6mm_W2.0mm_P2.50mm_MKS02_FKP02, F.Cu at (135.0, 90.2)
- added C2: 100nF, Capacitor_THT:C_Rect_L4.6mm_W2.0mm_P2.50mm_MKS02_FKP02, F.Cu at (117.8, 49.8)
- added C3: 100nF, Capacitor_THT:C_Rect_L4.6mm_W2.0mm_P2.50mm_MKS02_FKP02, F.Cu at (137.8, 38.2)
- added C7: 100nF, Capacitor_THT:C_Rect_L4.6mm_W2.0mm_P2.50mm_MKS02_FKP02, F.Cu at (117.2, 36.9)
- added D1: YELLOW, LED_THT:LED_D5.0mm, F.Cu at (98.9, 90.4)
- added J1: 1MHz CLK, Connector_PinHeader_2.54mm:PinHeader_1x02_P2.54mm_Vertical, F.Cu at (141.7, 68.9)
- added J3: Barrel_Jack_Switch, Connector_BarrelJack:BarrelJack_Kycon_KLDX-0202-xC_Horizontal, F.Cu at (135.1, 31.8)
- added J4: PWR IN, Connector_PinSocket_2.54mm:PinSocket_1x02_P2.54mm_Vertical, F.Cu at (131.0, 29.2)
- added J5: Universal Bus Connector v2, Connector_PinSocket_2.54mm:PinSocket_1x18_P2.54mm_Vertical, F.Cu at (121.6, 40.0)
- added J6: Universal Bus Connector v2, Connector_PinSocket_2.54mm:PinSocket_1x18_P2.54mm_Vertical, F.Cu at (121.6, 80.0)
- added R1: 1k, Resistor_THT:R_Axial_DIN0207_L6.3mm_D2.5mm_P10.16mm_Horizontal, F.Cu at (131.9, 89.7)
- added R8: 220, Resistor_THT:R_Axial_DIN0207_L6.3mm_D2.5mm_P10.16mm_Horizontal, F.Cu at (95.1, 90.8)
- added SW1: Push, Button_Switch_THT:SW_PUSH_6mm, F.Cu at (122.0, 93.3)
- added U1: W65C02SxP, Package_DIP:DIP-40_W15.24mm, F.Cu at (135.6, 52.3)
- added Y1: ACO-xxxMHz, Oscillator:Oscillator_DIP-14, F.Cu at (146.8, 91.6)
Routing:
- net +5V: track 0.00 -> 188.5 mm
- net Net-(J6-Pin_15): track 0.00 -> 150.8 mm
- net Net-(J6-Pin_16): track 0.00 -> 141.1 mm
- net Net-(J6-Pin_17): track 0.00 -> 132.8 mm
- net Net-(J6-Pin_18): track 0.00 -> 124.8 mm
- net Net-(J6-Pin_12): track 0.00 -> 74.2 mm
- net Net-(J1-Pin_1): track 0.00 -> 67.1 mm
- net Net-(J5-Pin_15): track 0.00 -> 49.2 mm
- net Net-(J5-Pin_16): track 0.00 -> 45.2 mm
- net Net-(J5-Pin_17): track 0.00 -> 41.3 mm
- net Net-(J5-Pin_18): track 0.00 -> 36.0 mm
- net Net-(J6-Pin_1): track 0.00 -> 14.1 mm
- net Net-(J6-Pin_2): track 0.00 -> 13.0 mm
- net Net-(J6-Pin_9): track 0.00 -> 13.0 mm
- net Net-(J6-Pin_7): track 0.00 -> 13.0 mm
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- added copper zone on B.Cu, net GND
Other:
- board outline added: 100 x 70 mm
- copper layers 0 -> 2

Commit message: 28c256 rom pcb
Parts:
- added C8: 100nF, Capacitor_THT:C_Rect_L4.6mm_W2.0mm_P2.50mm_MKS02_FKP02, F.Cu at (88.5, 76.9)
- J5: value Universal Bus Connector v2 -> Universal Bus Connector A
- J6: value Universal Bus Connector v2 -> Universal Bus Connector B
Routing:
- net +5V: track 188.5 -> 191.7 mm
