File: 6502-pcbs/6502-mainboard/6502-mainboard.kicad_sch (KiCad schematic)
At the start: 0 parts

Commit message: 6502 mainboard
Parts:
- added C1: 10uF+, Capacitor_THT:CP_Radial_D7.5mm_P2.50mm, symbol Device:C_Polarized_Small
- added C13, C2, C3, C7: 100nF, Capacitor_THT:C_Rect_L4.6mm_W2.0mm_P2.50mm_MKS02_FKP02, symbol Device:C_Small
- added D1: YELLOW, LED_THT:LED_D5.0mm, symbol Device:LED
- added J1: 1MHz CLK, Connector_PinHeader_2.54mm:PinHeader_1x02_P2.54mm_Vertical, symbol Connector_Generic:Conn_01x02
- added J3: Barrel_Jack_Switch, Connector_BarrelJack:BarrelJack_Kycon_KLDX-0202-xC_Horizontal, symbol Connector:Barrel_Jack_Switch
- added J4: PWR IN, Connector_PinSocket_2.54mm:PinSocket_1x02_P2.54mm_Vertical, symbol Connector_Generic:Conn_01x02
- added J5, J6: Universal Bus Connector v2, Connector_PinSocket_2.54mm:PinSocket_1x18_P2.54mm_Vertical, symbol Connector:Conn_01x18_Socket
- added R1: 1k, Resistor_THT:R_Axial_DIN0207_L6.3mm_D2.5mm_P10.16mm_Horizontal, symbol Device:R_Small_US
- added R8: 220, Resistor_THT:R_Axial_DIN0207_L6.3mm_D2.5mm_P10.16mm_Horizontal, symbol Device:R_Small_US
- added SW1: Push, Button_Switch_THT:SW_PUSH_6mm, symbol Switch:SW_Push
- added U1: W65C02SxP, Package_DIP:DIP-40_W15.24mm, symbol 65xx-library:W65C02SxP
- added Y1: ACO-xxxMHz, Oscillator:Oscillator_DIP-14, symbol Oscillator:ACO-xxxMHz
Connections:
- new net: J6.12 (Pin_12), R1.2, SW1.2, U1.40 (~{RES})
- new net: J1.1 (Pin_1), J6.11 (Pin_11), U1.37 (ϕ0)
- new net: J1.2 (Pin_2), Y1.8 (OUT)
- new net: D1.1 (K), R8.1
- new net: J5.4 (Pin_4), U1.10 (A1)
- new net: J5.5 (Pin_5), U1.11 (A2)
- new net: J5.6 (Pin_6), U1.12 (A3)
- new net: J5.7 (Pin_7), U1.13 (A4)
- new net: J5.8 (Pin_8), U1.14 (A5)
- new net: J5.9 (Pin_9), U1.15 (A6)
- new net: J5.10 (Pin_10), U1.16 (A7)
- new net: J5.11 (Pin_11), U1.17 (A8)
- new net: J5.12 (Pin_12), U1.18 (A9)
- new net: J5.13 (Pin_13), U1.19 (A10)
- new net: J6.15 (Pin_15), U1.2 (RDY)
- new net: J5.14 (Pin_14), U1.20 (A11)
- new net: J5.15 (Pin_15), U1.22 (A12)
- new net: J5.16 (Pin_16), U1.23 (A13)
- new net: J5.17 (Pin_17), U1.24 (A14)
- new net: J5.18 (Pin_18), U1.25 (A15)
- new net: J6.10 (Pin_10), U1.26 (D7)
- new net: J6.9 (Pin_9), U1.27 (D6)
- new net: J6.8 (Pin_8), U1.28 (D5)
- new net: J6.7 (Pin_7), U1.29 (D4)
- new net: J6.6 (Pin_6), U1.30 (D3)
- new net: J6.5 (Pin_5), U1.31 (D2)
- new net: J6.4 (Pin_4), U1.32 (D1)
- new net: J6.3 (Pin_3), U1.33 (D0)
- new net: J6.2 (Pin_2), U1.34 (R/~{W})
- new net: J6.1 (Pin_1), U1.36 (BE)
- new net: J6.16 (Pin_16), U1.4 (~{IRQ})
- new net: J6.17 (Pin_17), U1.6 (~{NMI})
- new net: J6.18 (Pin_18), U1.7 (SYNC)
- new net: J5.3 (Pin_3), U1.9 (A0)
- new net +5V: C1.1, C13.1, C2.1, C3.1, C7.1, D1.2 (A), J3.1, J4.2 (Pin_2), J5.2 (Pin_2), J6.13 (Pin_13), R1.1, U1.38 (~{SO}), U1.8 (VDD), Y1.14 (Vcc)
- new net GND: C1.2, C13.2, C2.2, C3.2, C7.2, J3.2, J3.3, J4.1 (Pin_1), J5.1 (Pin_1), J6.14 (Pin_14), R8.2, SW1.1, U1.21 (VSS), Y1.7 (GND)
- no-connect marks 0 -> 4
Other:
- company: (none) -> Sam Warr
- title: (none) -> 6502 Mainboard

Commit message: 28c256 rom pcb
Parts:
- added C8: 100nF, Capacitor_THT:C_Rect_L4.6mm_W2.0mm_P2.50mm_MKS02_FKP02, symbol Device:C_Small
Connections:
- net +5V: now also C8.2
- net GND: now also C8.1
Other:
- moved on the sheet: J4
