File: 6502-pcbs/universal-bus-connector/universal-bus-connector.kicad_sch (KiCad schematic)
At the start: 5 parts, among them J1 Universal Bus Connector v2, J2 Universal Bus Connector v2, J3 Universal Bus Connector v2, J4 Universal Bus Connector v2

Commit message: 28c256 rom
Parts:
- J1, J3: value Universal Bus Connector v2 -> Universal Bus Connector
Connections:
- net +5V: now also J4.13 (Pin_13)
- net GND: now also J4.14 (Pin_14)
Changed lines of the file:
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@@
+	(wire
+		(pts
+			(xy 129.54 71.12) (xy 130.81 71.12)
+		)
+		(stroke
+			(width 0)
+			(type default)
+		)
+	)
 	(wire
 		(pts
@@
 		(pts
 			(xy 114.3 43.18) (xy 116.84 43.18)
+		)
+		(stroke
+			(width 0)
+			(type default)
+		)
+	)
+	(wire
+		(pts
+			(xy 129.54 73.66) (xy 130.81 73.66)
 		)
 		(stroke
@@
 			)
 		)
-		(property "Value" "Universal Bus Connector v2"
+		(property "Value" "Universal Bus Connector"
 			(at 110.49 36.576 0)
 			(effects
@@
 			)
 		)
-		(property "Value" "Universal Bus Connector v2"
+		(property "Value" "Universal Bus Connector"
 			(at 72.39 36.576 0)
 			(effects
@@
 				(path "/120d2c49-daff-425e-8ff2-b09f7f99bbee"
 					(reference "J1")
+					(unit 1)
+				)
+			)
+		)
+	)
+	(symbol
+		(lib_id "power:GND")
+		(at 130.81 73.66 0)
+		(unit 1)
+		(body_style 1)
+		(exclude_from_sim no)
+		(in_bom yes)
+		(on_board yes)
+		(dnp no)
+		(property "Reference" "#PWR06"
+			(at 130.81 80.01 0)
+			(hide yes)
+			(effects
+				(font
+					(size 1.27 1.27)
+				)
+			)
+		)
+		(property "Value" "GND"
+			(at 135.128 75.184 0)
+			(effects
+				(font
+					(size 1.27 1.27)
+				)
+			)
+		)
+		(property "Footprint" ""
+			(at 130.81 73.66 0)
+			(hide yes)
+			(effects
+				(font
+					(size 1.27 1.27)
+				)
+			)
+		)
+		(property "Datasheet" ""
+			(at 130.81 73.66 0)
+			(hide yes)
+			(effects
+				(font
+					(size 1.27 1.27)
+				)
+			)
+		)
+		(property "Description" "Power symbol creates a global label with name \"GND\" , ground"
+			(at 130.81 73.66 0)
+			(hide yes)
+			(effects
+				(font
+					(size 1.27 1.27)
+				)
+			)
+		)
+		(pin "1"
+		)
+		(instances
+			(project "universal-bus-connector"
+				(path "/120d2c49-daff-425e-8ff2-b09f7f99bbee"
+					(reference "#PWR06")
 					(unit 1)
 				)
@@
 					(unit 1)
 				)
+			)
+		)
+	)
+	(symbol
+		(lib_id "power:+5V")
+		(at 130.81 71.12 0)
+		(unit 1)
+		(body_style 1)
+		(exclude_from_sim no)
+		(in_bom yes)
+		(on_board yes)
+		(dnp no)
+		(property "Reference" "#PWR05"
+			(at 130.81 74.93 0)
+			(hide yes)
+			(effects
+				(font
+					(size 1.27 1.27)
+				)
+			)
+		)
+		(property "Value" "+5V"
+			(at 132.842 69.342 0)
+			(effects
+				(font
+					(size 1.27 1.27)
+				)
+			)
+		)
+		(property "Footprint" ""
+			(at 130.81 71.12 0)
+			(hide yes)
+			(effects
+				(font
+					(size 1.27 1.27)
+				)
+			)
+		)
+		(property "Datasheet" ""
+			(at 130.81 71.12 0)
+			(hide yes)
+			(effects
+				(font
+					(size 1.27 1.27)
+				)
+			)
+		)
+		(property "Description" "Power symbol creates a global label with name \"+5V\""
+			(at 130.81 71.12 0)
+			(hide yes)
+			(effects
+				(font
+					(size 1.27 1.27)
+				)
+			)
+		)
+		(pin "1"
+		)
+		(instances
+			(project "universal-bus-connector"
+				(path "/120d2c49-daff-425e-8ff2-b09f7f99bbee"
+					(reference "#PWR05")
+					(unit 1)
+				)

Commit message: 28c256 rom pcb
Parts:
- added C8: 100nF, Capacitor_THT:C_Rect_L4.6mm_W2.0mm_P2.50mm_MKS02_FKP02, symbol Device:C_Small
- J1, J3: value Universal Bus Connector -> Universal Bus Connector A
- J2, J4: value Universal Bus Connector v2 -> Universal Bus Connector B
Connections:
- net +5V: now also C8.2; no longer J4.2 (Pin_2)
- net GND: now also C8.1; no longer J4.1 (Pin_1)
Changed lines of the file:
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@@
+	)
+	(junction
+		(at 130.81 71.12)
+		(diameter 0)
+		(color 0 0 0 0)
 	)
 	(junction
@@
 		(color 0 0 0 0)
 	)
+	(junction
+		(at 130.81 73.66)
+		(diameter 0)
+		(color 0 0 0 0)
+	)
+	(wire
+		(pts
+			(xy 134.62 69.85) (xy 132.08 69.85)
+		)
+		(stroke
+			(width 0)
+			(type default)
+		)
+	)
+	(wire
+		(pts
+			(xy 132.08 73.66) (xy 130.81 73.66)
+		)
+		(stroke
+			(width 0)
+			(type default)
+		)
+	)
+	(wire
+		(pts
+			(xy 132.08 69.85) (xy 132.08 71.12)
+		)
+		(stroke
+			(width 0)
+			(type default)
+		)
+	)
 	(wire
 		(pts
@@
 	(wire
 		(pts
-			(xy 129.54 43.18) (xy 132.08 43.18)
+			(xy 114.3 44.45) (xy 114.3 43.18)
 		)
 		(stroke
@@
 	(wire
 		(pts
-			(xy 114.3 44.45) (xy 114.3 43.18)
+			(xy 129.54 71.12) (xy 130.81 71.12)
 		)
 		(stroke
@@
 	(wire
 		(pts
-			(xy 129.54 71.12) (xy 130.81 71.12)
+			(xy 132.08 74.93) (xy 132.08 73.66)
+		)
+		(stroke
+			(width 0)
+			(type default)
+		)
+	)
+	(wire
+		(pts
+			(xy 132.08 71.12) (xy 130.81 71.12)
+		)
+		(stroke
+			(width 0)
+			(type default)
+		)
+	)
+	(wire
+		(pts
+			(xy 134.62 74.93) (xy 132.08 74.93)
 		)
 		(stroke
@@
 				(path "/120d2c49-daff-425e-8ff2-b09f7f99bbee"
 					(reference "#PWR048")
+					(unit 1)
+				)
+			)
+		)
+	)
+	(symbol
+		(lib_id "Device:C_Small")
+		(at 134.62 72.39 0)
+		(mirror x)
+		(unit 1)
+		(body_style 1)
+		(exclude_from_sim no)
+		(in_bom yes)
+		(on_board yes)
+		(dnp no)
+		(property "Reference" "C8"
+			(at 134.874 71.12 0)
+			(effects
+				(font
+					(size 1.27 1.27)
+				)
+				(justify right)
+			)
+		)
+		(property "Value" "100nF"
+			(at 137.16 73.914 0)
+			(effects
+				(font
+					(size 1.27 1.27)
+				)
+				(justify right)
+			)
+		)
+		(property "Footprint" "Capacitor_THT:C_Rect_L4.6mm_W2.0mm_P2.50mm_MKS02_FKP02"
+			(at 134.62 72.39 0)
+			(hide yes)
+			(effects
+				(font
+					(size 1.27 1.27)
+				)
+			)
+		)
+		(property "Datasheet" ""
+			(at 134.62 72.39 0)
+			(hide yes)
+			(effects
+				(font
+					(size 1.27 1.27)
+				)
+			)
+		)
+		(property "Description" "Unpolarized capacitor, small symbol"
+			(at 134.62 72.39 0)
+			(hide yes)
+			(effects
+				(font
+					(size 1.27 1.27)
+				)
+			)
+		)
+		(pin "1"
+		)
+		(pin "2"
+		)
+		(instances
+			(project "universal-bus-connector"
+				(path "/120d2c49-daff-425e-8ff2-b09f7f99bbee"
+					(reference "C8")
 					(unit 1)
 				)
@@
 			)
 		)
-		(property "Value" "Universal Bus Connector v2"
+		(property "Value" "Universal Bus Connector B"
 			(at 125.984 36.576 0)
 			(hide yes)
@@
 			)
 		)
-		(property "Value" "Universal Bus Connector"
+		(property "Value" "Universal Bus Connector A"
 			(at 110.49 36.576 0)
 			(effects
@@
 			)
 		)
-		(property "Value" "Universal Bus Connector v2"
+		(property "Value" "Universal Bus Connector B"
 			(at 87.884 36.576 0)
 			(hide yes)
@@
 				(path "/120d2c49-daff-425e-8ff2-b09f7f99bbee"
 					(reference "J2")
-					(unit 1)
-				)
-			)
-		)
-	)
-	(symbol
-		(lib_id "power:GND")
-		(at 129.54 40.64 0)
-		(mirror y)
-		(unit 1)
-		(body_style 1)
-		(exclude_from_sim no)
-		(in_bom yes)
-		(on_board yes)
-		(dnp no)
-		(property "Reference" "#PWR049"
-			(at 129.54 46.99 0)
-			(hide yes)
-			(effects
-				(font
-					(size 1.27 1.27)
-				)
-			)
-		)
-		(property "Value" "GND"
-			(at 129.54 41.148 0)
-			(effects
-				(font
-					(size 1.27 1.27)
-				)
-			)
-		)
-		(property "Footprint" ""
-			(at 129.54 40.64 0)
-			(hide yes)
-			(effects
-				(font
-					(size 1.27 1.27)
-				)
-			)
-		)
-		(property "Datasheet" ""
-			(at 129.54 40.64 0)
-			(hide yes)
-			(effects
-				(font
-					(size 1.27 1.27)
-				)
-			)
-		)
-		(property "Description" "Power symbol creates a global label with name \"GND\" , ground"
-			(at 129.54 40.64 0)
-			(hide yes)
-			(effects
-				(font
-					(size 1.27 1.27)
-				)
-			)
-		)
-		(pin "1"
-		)
-		(instances
-			(project "universal-bus-connector"
-				(path "/120d2c49-daff-425e-8ff2-b09f7f99bbee"
-					(reference "#PWR049")
 					(unit 1)
 				)
@@
 			)
 		)
-		(property "Value" "Universal Bus Connector"
-			(at 72.39 36.576 0)
+		(property "Value" "Universal Bus Connector A"
+			(at 71.374 36.322 0)
 			(effects
 				(font
@@
 		)
 		(property "Value" "GND"
-			(at 135.128 75.184 0)
+			(at 133.096 75.184 0)
 			(effects
 				(font
@@
 				(path "/120d2c49-daff-425e-8ff2-b09f7f99bbee"
 					(reference "#PWR06")
-					(unit 1)
-				)
-			)
-		)
-	)
-	(symbol
-		(lib_id "power:+5V")
-		(at 132.08 43.18 0)
-		(mirror y)
-		(unit 1)
-		(body_style 1)
-		(exclude_from_sim no)
-		(in_bom yes)
-		(on_board yes)
-		(dnp no)
-		(property "Reference" "#PWR039"
-			(at 132.08 46.99 0)
-			(hide yes)
-			(effects
-				(font
-					(size 1.27 1.27)
-				)
-			)
-		)
-		(property "Value" "+5V"
-			(at 132.334 42.164 0)
-			(effects
-				(font
-					(size 1.27 1.27)
-				)
-			)
-		)
-		(property "Footprint" ""
-			(at 132.08 43.18 0)
-			(hide yes)
-			(effects
-				(font
-					(size 1.27 1.27)
-				)
-			)
-		)
-		(property "Datasheet" ""
-			(at 132.08 43.18 0)
-			(hide yes)
-			(effects
-				(font
-					(size 1.27 1.27)
-				)
-			)
-		)
-		(property "Description" "Power symbol creates a global label with name \"+5V\""
-			(at 132.08 43.18 0)
-			(hide yes)
-			(effects
-				(font
-					(size 1.27 1.27)
-				)
-			)
-		)
-		(pin "1"
-		)
-		(instances
-			(project "universal-bus-connector"
-				(path "/120d2c49-daff-425e-8ff2-b09f7f99bbee"
-					(reference "#PWR039")
 					(unit 1)
 				)
@@
 		)
 		(property "Value" "+5V"
-			(at 132.842 69.342 0)
-			(effects
-				(font
+			(at 132.08 70.104 0)
+			(effects
+				(font
